File: LED-Driver-Breakout.kicad_pcb (KiCad board)
At the start: 6 copper layers, 98 x 100 mm, 27 parts, among them U1 V10P45-M3/86A, U2 TSR0.5-2418

Commit message: Added project-specific libs/fps; updates generally; broken rn.
Parts:
- removed  : MountingHole_3.2mm_M3_Pad_Via, MountingHole:MountingHole_3.2mm_M3_Pad_Via (x4)
- removed  : JST_XH_S2B-XH-A_1x02_P2.50mm_Horizontal, Connector_JST:JST_XH_S2B-XH-A_1x02_P2.50mm_Horizontal
- removed  : AMASS_XT60PW-M_1x02_P7.20mm_Horizontal, Connector_AMASS:AMASS_XT60PW-M_1x02_P7.20mm_Horizontal
- removed Analog-Dim, Batt+, GND (x2), Switch(PWM-Dim), V_Fused, V_Regulated: TestPoint_Loop_D1.80mm_Drill1.0mm_Beaded, TestPoint:TestPoint_Loop_D1.80mm_Drill1.0mm_Beaded
- removed REF**: PinHeader_1x02_P1.00mm_Vertical, Connector_PinHeader_1.00mm:PinHeader_1x02_P1.00mm_Vertical
- removed REF**: TerminalBlock_WAGO_2601-1102_1x02_P3.50mm_Horizontal, TerminalBlock_WAGO:TerminalBlock_WAGO_2601-1102_1x02_P3.50mm_Horizontal
- added C6: 10 µF, Capacitor_SMD:C_0805_2012Metric_Pad1.18x1.45mm_HandSolder, F.Cu at (-45.6, 127.8)
- added J1: S2B-XH-A, Project_Footprints_Lib:JST_XH_S2B-XH-A_1x02_P2.50mm_Horizontal, F.Cu at (79.4, 70.1)
- added J2: LED Output, TerminalBlock_WAGO:TerminalBlock_WAGO_2601-3102_1x02_P3.50mm_Vertical, F.Cu at (76.3, 84.0)
- C1: footprint Capacitor_SMD:C_0805_2012Metric_Pad1.18x1.45mm_HandSolder -> Project_Footprints_Lib:C_0805_2012Metric_Pad1.18x1.45mm_HandSolder
- F1: footprint KiCad333:154005DR -> Project_Footprints_Lib:154005DR
- PS1: footprint KiCad:LDH45B1050 -> Project_Footprints_Lib:LDH-45B-1050
- U2: value TSR0.5-2418 -> TSR2-24120; footprint Converter_DCDC:Converter_DCDC_TRACO_TSR0.5-24xx_TSR0.5-24xxx_THT -> Converter_DCDC:Converter_DCDC_TRACO_TSR2-xxxx_THT
- moved C5 205.3 mm to (-53.8, 125.2), turned to 0 degrees
- moved C4 197.7 mm to (-45.6, 124.8), turned to 0 degrees
- moved C3 197.6 mm to (-45.6, 121.8), turned to 0 degrees
- moved C1 193.4 mm to (-18.4, 172.0)
- moved C2 193.4 mm to (-11.2, 172.0)
- moved L1 192.1 mm to (-40.8, 127.3), turned to 0 degrees
- moved F1 146.2 mm to (23.8, 144.2)
- moved U1 141.4 mm to (46.9, 163.2), turned to 90 degrees
- moved R1 137.3 mm to (21.1, 123.2)
- moved D1 136.2 mm to (27.2, 123.0)
- moved U2 73.5 mm to (91.4, 75.2), turned to 180 degrees
- moved PS1 23.6 mm to (137.6, 88.5), turned to -90 degrees
Connections:
- C1 pad 1: V_Fused -> /V_Fused
- C1 pad 2: GND -> Net-(PS1-VIN-)
- C2 pad 1: V_Fused -> /V_Fused
- C2 pad 2: GND -> Net-(PS1-VIN-)
- C3 pad 1: V_Fused -> /V_Fused
- C3 pad 2: GND -> Net-(U2-GND)
- C4 pad 1: V_Fused -> /V_Fused
- C4 pad 2: GND -> Net-(U2-GND)
- C5 pad 2: GND -> Net-(U2-GND)
- D1 pad 1: GND -> /GND
- F1 pad 1: +BATT -> Net-(F1-Pad1)
- L1 pad 1: V_Fused -> /V_Fused
- PS1 pad 1: V_Fused -> /V_Fused
- PS1 pad 2: GND -> Net-(PS1-VIN-)
- PS1 pad 3: GND -> /GND
- PS1 pad 6: VOUT- -> Net-(PS1-VOUT-)
- PS1 pad 7: VOUT+ -> Net-(PS1-VOUT+)
- R1 pad 1: V_Fused -> /V_Fused
- U1 pad 1: Net-(F1-Pad2) -> /V_Fused
- U2 pad 2: GND -> Net-(U2-GND)
- U2 pad 3: VRegulated -> Net-(U2-Vout)
Routing:
- net +BATT: track 99.4 -> 0.00 mm
- net /switch: track 79.2 -> 0.00 mm
- net GND: track 57.4 -> 0.00 mm, vias 3 -> 0
- net VOUT+: track 38.9 -> 0.00 mm
- net Net-(PS1-VOUT+): track 0.00 -> 38.9 mm
- net V_Fused: track 36.7 -> 0.00 mm, vias 4 -> 0
- net unconnected-(PS1-ANALOG_DIM-Pad4): track 35.0 -> 0.00 mm
- net VOUT-: track 24.7 -> 0.00 mm
- net Net-(PS1-VOUT-): track 0.00 -> 24.7 mm
- net Net-(U2-Vin): track 22.9 -> 0.00 mm
- net Net-(F1-Pad2): track 11.1 -> 0.00 mm
- net Net-(D1-A): track 5.03 -> 0.00 mm
- added copper zone on In1.Cu, net /GND
- added copper zone on In4.Cu, net /GND
- added copper zone on In2.Cu, net /V_Fused
- added copper zone on In3.Cu, net Net-(U2-Vout)
- removed copper zone on In1.Cu, net GND
- removed copper zone on In4.Cu, net GND
- removed copper zone on In3.Cu, net VRegulated
- removed copper zone on In2.Cu, net V_Fused
Other:
- board text removed: "5A Fuse"
- board text removed: "Switch (PWM-Dim)"

Commit message: Relayout in progress.
Parts:
- added J3: XT60, Connector_AMASS:AMASS_XT60PW-M_1x02_P7.20mm_Horizontal, F.Cu at (85.2, 73.6)
- added J4: 01x03_PinHeaderSwitch, Connector_PinHeader_2.54mm:PinHeader_1x03_P2.54mm_Vertical, F.Cu at (79.4, 108.4)
- moved C5 155.8 mm to (98.5, 92.3), turned to 180 degrees
- moved C3 141.6 mm to (94.9, 104.8)
- moved C4 141.6 mm to (94.9, 107.8)
- moved C6 141.6 mm to (94.9, 110.8)
- moved L1 141.6 mm to (99.8, 110.2)
- moved C1 120.1 mm to (94.9, 132.1)
- moved C2 120.1 mm to (102.1, 132.1)
- moved U1 113.9 mm to (100.6, 62.7)
- moved F1 106.6 mm to (92.8, 63.1), turned to 90 degrees
- moved D1 71.5 mm to (98.7, 120.3)
- moved R1 71.5 mm to (92.5, 120.6)
- moved U2 15.1 mm to (89.2, 90.1)
- moved J2 14.5 mm to (75.3, 98.5)
- moved J1 14.2 mm to (78.4, 84.3)
- moved PS1 0.76 mm to (137.2, 87.8)
Routing:
- net /V_Fused: track 0.04 -> 58.5 mm
- net Net-(PS1-VOUT+): track 38.9 -> 13.7 mm
- net Net-(PS1-VOUT-): track 24.7 -> 0.00 mm
- net Net-(F1-Pad2): track 0.00 -> 8.99 mm
- net Net-(F1-Pad1): track 0.00 -> 7.65 mm
